File: ZX Spectrum AMP.kicad_sch (KiCad schematic)
At the start: 13 parts, among them IC1 LM386, J1 9V DC(in), J2 Input (MIC), J3 9V DC(out), P1 4,7K Ohm

Commit message: updated
Parts:
- added H1, H2, H3, H4: MountingHole, MountingHole:MountingHole_3.5mm, symbol Mechanical:MountingHole
- added P2: 50K, Potentiometer_THT:Potentiometer_Piher_PT-10-V10_Vertical, symbol Device:R_Potentiometer
- P1: value 4,7K Ohm -> 4.7K
- R1: value 10 Ohm -> 10
Connections:
- net GND: now also P2.3
- net at MIC1.1 (Pin_1), P1.1: now also P2.1; no longer J2.1
- new net: J2.1, P2.2
Other:
- note added: "Mounting holes"
- company: (none) -> Ny Elektronik
- title: (none) -> ZX Spectrum Amplifier
- moved on the sheet: J2, MIC1
